Commit message: Added MoveIt motion planning from detected cube positions

File: src/so101_description/urdf/so101_new_calib.urdf (robot description, URDF)
Before this commit: robot so101_new_calib, 8 links, 7 joints
Links:
- link base_link: geometry collision mesh filename=package://so101_description/assets/base_motor_holder_so101_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; collision mesh filename=package://so101_description/assets/base_so101_v2.stl
- link gripper_link: geometry collision mesh filename=package://so101_description/assets/sts3215_03a_v1.stl; collision mesh filename=package://so101_description/assets/wrist_roll_follower_so10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
- link lower_arm_link: geometry collision mesh filename=package://so101_description/assets/motor_holder_so101_wrist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; collision mesh filename=package://so101_description/assets/sts3215_03a_v1.stl
- link moving_jaw_so101_v1_link: geometry collision mesh filename=package://so101_description/assets/moving_jaw_so101_v1.stl; visual mesh filename=package://so101_description/assets/moving_jaw_so101_v1.stl
- link shoulder_link: geometry collision mesh filename=package://so101_description/assets/motor_holder_so101_base_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; collision mesh filename=package://so101_description/assets/rotation_pitch_so101_v1.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
- link upper_arm_link: geometry collision mesh filename=package://so101_description/assets/sts3215_03a_v1.stl; collision mesh filename=package://so101_description/assets/upper_arm_so101_v1.stl
- link wrist_link: geometry collision mesh filename=package://so101_description/assets/sts3215_03a_no_horn_v1.s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; collision mesh filename=package://so101_description/assets/wrist_roll_pitch_so101_v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

File: src/so101_description/urdf/so101_scene.urdf.xacro (robot description, xacro)
@@ -1,5 +1,5 @@
 <?xml version="1.0"?>
 <robot name="so101_scene" xmlns:xacro="http://www.ros.org/wiki/xacro">
-  <xacro:include filename="$(find arm_description)/urdf/so101_new_calib.urdf"/>
+  <xacro:include filename="$(find so101_description)/urdf/so101_new_calib.urdf"/>
   <xacro:property name="table_x"     value="1.0"/>
   <xacro:property name="table_y"     value="0.6"/>
