Commit message: fixed urdf

File: src/so101_description/urdf/dual_arm_final.urdf.xacro (robot description, xacro)
@@ -15,12 +15,12 @@
   <xacro:property name="leg_length"  value="${table_top_z - table_thick}"/>
   <!-- ================= ROBOTS =================== -->
-  <xacro:property name="robot_y"       value="${table_y/2}"/>
+  <xacro:property name="robot_y"       value="${(table_y/2)-0.015}"/>
   <xacro:property name="robot_left_x"  value="-0.25"/>
   <xacro:property name="robot_right_x" value="0.25"/>
   <xacro:property name="robot_yaw"     value="${-pi/2}"/>
   <!-- ================= CAMERA ================= -->
-  <xacro:property name="pipe_radius" value="0.02"/>
-  <xacro:property name="pipe_length" value="0.65"/>
-  <xacro:property name="pipe_x" value="0.0"/>
+  <xacro:property name="pipe_radius" value="0.04"/>
+  <xacro:property name="pipe_length" value="0.58"/>
+  <xacro:property name="pipe_x" value="0.025"/>
   <xacro:property name="pipe_y" value="${robot_y}"/>
   <xacro:property name="cam_pitch" value="${pi/3}"/>

Commit message: modified urdfs

File: src/so101_description/urdf/dual_arm_final.urdf.xacro (robot description, xacro)
@@ -15,5 +15,5 @@
   <xacro:property name="leg_length"  value="${table_top_z - table_thick}"/>
   <!-- ================= ROBOTS =================== -->
-  <xacro:property name="robot_y"       value="${(table_y/2)-0.015}"/>
+  <xacro:property name="robot_y"       value="${(table_y/2) + 0.015}"/>
   <xacro:property name="robot_left_x"  value="-0.25"/>
   <xacro:property name="robot_right_x" value="0.25"/>
@@ -23,5 +23,5 @@
   <xacro:property name="pipe_length" value="0.58"/>
   <xacro:property name="pipe_x" value="0.025"/>
-  <xacro:property name="pipe_y" value="${robot_y}"/>
+  <xacro:property name="pipe_y" value="${(table_y/2)}"/>
   <xacro:property name="cam_pitch" value="${pi/3}"/>
   <xacro:property name="cam_yaw"   value="${-pi/2}"/>
@@ -119,5 +119,5 @@
     <parent link="table_link"/>
     <child link="upper_shelf_link"/>
-    <origin xyz="0 ${shelf_y_pos} 0" rpy="0 0 0"/>
+    <origin xyz="0 ${(shelf_y_pos)} 0" rpy="0 0 0"/>
   </joint>
   <!-- ================= PILLARS ================= -->
@@ -186,5 +186,5 @@
   <link name="camera_mount_link">
     <visual>
-      <origin xyz="0 0 0" rpy="0 0 0"/>
+      <origin xyz="0.06 0 0" rpy="0 0 0"/>
       <geometry>
         <box size="0.14 0.015 0.05"/>
@@ -195,5 +195,5 @@
       <origin xyz="0.06 0 0" rpy="0 0 0"/>
       <geometry>
-        <box size="0.12 0.015 0.015"/>
+        <box size="0.14 0.015 0.05"/>
       </geometry>
     </collision>
@@ -202,5 +202,5 @@
     <parent link="pipe_link"/>
     <child link="camera_mount_link"/>
-    <origin xyz="0 0 ${pipe_length}" rpy="0 0 0"/>
+    <origin xyz="0 -0.025 ${pipe_length}" rpy="0 0 0"/>
   </joint>
   <!-- ================= CAMERA ================= -->
@@ -221,5 +221,5 @@
     <parent link="camera_mount_link"/>
     <child link="camera_link"/>
-    <origin xyz="0 -0.015 0" rpy="0 ${cam_pitch} ${cam_yaw}"/>
+    <origin xyz="0 -0.017 0" rpy="0 ${cam_pitch} ${cam_yaw}"/>
   </joint>
   <!-- ================= OPTICAL FRAME ================= -->

Commit message: Add bin model to workspace URDF

File: src/so101_description/urdf/dual_arm_final.urdf.xacro (robot description, xacro)
@@ -36,4 +36,10 @@
   <!-- opposite side of robots -->
   <xacro:property name="shelf_y_pos" value="${-table_y/2 + shelf_y/2}"/>
+  <!-- ================= BIN ================= -->
+  <xacro:property name="bin_size" value="0.127"/>
+  <xacro:property name="bin_height" value="0.06"/>
+  <!-- centered between robots, slightly in front of camera pole -->
+  <xacro:property name="bin_x" value="0.0"/>
+  <xacro:property name="bin_y" value="0.15"/>
   <!-- ================= MATERIALS ================= -->
   <material name="wood">
@@ -51,4 +57,7 @@
   <material name="sts3215">
     <color rgba="0.1 0.1 0.1 1.0"/>
+  </material>
+  <material name="bin_orange">
+    <color rgba="1.0 0.5 0.0 1.0"/>
   </material>
   <!-- ================= WORLD ================= -->
@@ -230,3 +239,51 @@
     <origin xyz="0 0 0" rpy="${-pi/2} 0 ${-pi/2}"/>
   </joint>
+  <!-- ================= BIN ================= -->
+  <link name="bin_link">
+    <!-- Bottom -->
+    <visual>
+    <origin xyz="0 0 0.0025"/>
+    <geometry>
+      <box size="0.1 0.1 0.005"/>
+    </geometry>
+    <material name="bin_orange"/>
+    </visual>
+    <!-- Front wall -->
+    <visual>
+      <origin xyz="0 0.0525 0.03"/>
+      <geometry>
+        <box size="0.110 0.005 0.06"/>
+      </geometry>
+      <material name="bin_orange"/>
+    </visual>
+    <!-- Back wall -->
+    <visual>
+      <origin xyz="0 -0.0525 0.03"/>
+      <geometry>
+        <box size="0.110 0.005 0.06"/>
+      </geometry>
+      <material name="bin_orange"/>
+    </visual>
+    <!-- Left wall -->
+    <visual>
+      <origin xyz="-0.0525 0 0.03"/>
+      <geometry>
+        <box size="0.005 0.1 0.06"/>
+      </geometry>
+      <material name="bin_orange"/>
+    </visual>
+    <!-- Right wall -->
+    <visual>
+      <origin xyz="0.0525 0 0.03"/>
+      <geometry>
+        <box size="0.005 0.1 0.06"/>
+      </geometry>
+      <material name="bin_orange"/>
+    </visual>
+  </link>
+  <joint name="shelf_to_bin" type="fixed">
+    <parent link="upper_shelf_link"/>
+    <child link="bin_link"/>
+    <origin xyz="0 0 0.13" rpy="0 0 0"/>
+  </joint>
 </robot>

Commit message: Fix pick-and-place sequence to release cube at bin

File: src/so101_description/urdf/dual_arm_final.urdf.xacro (robot description, xacro)
@@ -285,5 +285,5 @@
     <parent link="upper_shelf_link"/>
     <child link="bin_link"/>
-    <origin xyz="0 0 0.13" rpy="0 0 0"/>
+    <origin xyz="0.25 0 0.13" rpy="0 0 0"/>
   </joint>
 </robot>
